File: fiftyseven.sch (KiCad schematic (older format))
At the start: 105 parts, among them J1 Pins, J2 USB-C, J3 ESP32 JTAG, J4 ESP32 SERIAL, J5 STM32 SWD, J6 240x320_8bit, Q1 SS8050-G, Q2 SS8050-G, SW0:0 SW_Push, SW0:1 SW_Push, SW0:10 SW_Push, SW0:11 SW_Push, SW0:12 SW_Push, SW0:2 SW_Push, SW0:3 SW_Push, SW0:4 SW_Push, SW0:5 SW_Push, SW0:6 SW_Push, SW0:7 SW_Push, SW0:8 SW_Push, SW0:9 SW_Push, SW1 SW_SPST, SW1:0 SW_Push, SW1:1 SW_Push, SW1:10 SW_Push, SW1:11 SW_Push, SW1:12 SW_Push, SW1:2 SW_Push, SW1:3 SW_Push, SW1:4 SW_Push, SW1:5 SW_Push, SW1:6 SW_Push, SW1:7 SW_Push, SW1:8 SW_Push, SW1:9 SW_Push, SW2:0 SW_Push, SW2:1 SW_Push, SW2:10 SW_Push, SW2:11 SW_Push, SW2:2 SW_Push, SW2:3 SW_Push, SW2:4 SW_Push, SW2:5 SW_Push, SW2:6 SW_Push, SW2:7 SW_Push, SW2:8 SW_Push, SW2:9 SW_Push, SW3:0 SW_Push, SW3:1 SW_Push, SW3:10 SW_Push, SW3:11 SW_Push, SW3:12 SW_Push, SW3:2 SW_Push, SW3:3 SW_Push, SW3:4 SW_Push, SW3:5 SW_Push, SW3:6 SW_Push, SW3:7 SW_Push, SW3:8 SW_Push, SW3:9 SW_Push, SW4:0 SW_Push, SW4:1 SW_Push, SW4:2 SW_Push, SW4:3 SW_Push, SW4:4 SW_Push, U1 STM32G071RB, U2 ESP32 WROVER, U3 MCP73123, U4 MAX40200, U5 LTC3246

Commit message: updates
Parts:
- removed C14, C9: 10uF, Capacitors_SMD:C_0603, symbol Device:C
- removed C8: 2.2uF, Capacitors_SMD:C_0603, symbol Device:C
- removed J6: 240x320_8bit, seventykeys:LCD-320x240, symbol 240x320_8bit:240x320_8bit
- removed R8: 10k, Resistors_SMD:R_0603, symbol Device:R
- removed U4: MAX40200, TO_SOT_Packages_SMD:SOT-23-5, symbol MAX40200:MAX40200
- removed U5: LTC3246, seventykeys:MSOP-16-1EP-VIA_3x4mm_Pitch0.5mm, symbol LTC3246:LTC3246
- added R1: 10k, Resistors_SMD:R_0603, symbol Device:R
- added U4: LP5912, fiftyseven:LP5912, symbol LP5912:LP5912
- added U6: 240x320_16bit, fiftyseven:LCD-320x240, symbol 240x320_16bit:240x320_16bit
- BT1: footprint seventykeys:AA-clip -> fiftyseven:AA-clip
- C6: value 1uF -> 2.2uF
- C7: value 10uF -> 2.2uF; Comment Minimum 2uF -> Minimum 1uF
- SW0:0, SW0:1, SW0:10, SW0:11, SW0:12, SW0:2, SW0:3, SW0:4, SW0:5, SW0:6, SW0:7, SW0:8, SW0:9, SW1:0, SW1:1, SW1:10, SW1:11, SW1:12, SW1:2, SW1:3, SW1:4, SW1:5, SW1:6, SW1:7, SW1:8, SW1:9, SW2:0, SW2:1, SW2:10, SW2:11, SW2:2, SW2:3, SW2:4, SW2:5, SW2:6, SW2:7, SW2:8, SW2:9, SW3:0, SW3:1, SW3:10, SW3:11, SW3:12, SW3:2, SW3:3, SW3:4, SW3:5, SW3:6, SW3:7, SW3:8, SW3:9, SW4:0, SW4:1, SW4:2, SW4:3, SW4:4, SW:ESC1: footprint seventykeys:4.5mm-switch -> fiftyseven:4.5mm-switch
- SW1: value SW_SPST -> on/off switch; footprint seventykeys:on-off-switch -> fiftyseven:on-off-switch
- U1: footprint seventykeys:STM32G0-LQFP-64 -> fiftyseven:STM32G0-LQFP-64
- U2: footprint seventykeys:ESP32-WROVER -> fiftyseven:ESP32-WROVER
- U3: footprint seventykeys:MCP73123 -> fiftyseven:MCP73123
Connections:
- net +3V3 is gone; now on net +3V0: C1.2, C10.1, C11.1, C12.1, C13.1, C15.2, C16.2, C2.2, J1.19 (Pin_19), J1.2 (Pin_2), J3.1 (VCC), J4.1 (Pin_1), J5.1 (VCC), R10.1, R11.1, SW:ESC1.1, U1.6 (VBAT), U1.7 (VREF+), U1.8 (VDD/VDDA), U2.2 (3V3)
- net ~RST~ is gone; now on net PG: C17.1, C3.1, J3.10 (~RESET~), J4.7 (Pin_7), J5.10 (~RESET~), Q1.3 (C), U1.12 (PF2-NRST), U2.3 (EN)
- net C0: now also U1.13 (PC0); no longer U1.59 (PB5)
- net C1: now also U1.14 (PC1); no longer U1.58 (PB4)
- net C10: now also U1.1 (PC11); no longer U1.49 (PC9)
- net C11: now also U1.2 (PC12); no longer U1.48 (PC8)
- net C12: now also U1.3 (PC13); no longer U1.39 (PC7)
- net C2: now also U1.15 (PC2); no longer U1.57 (PB3)
- net C3: now also U1.16 (PC3); no longer U1.56 (PD6)
- net C4: now also U1.38 (PC6); no longer U1.55 (PD5)
- net C5: now also U1.39 (PC7); no longer U1.54 (PD4)
- net C6: now also U1.48 (PC8); no longer U1.53 (PD3)
- net C7: now also U1.41 (PD9); no longer U1.52 (PD2)
- net C8: now also U1.49 (PC9); no longer U1.51 (PD1)
- net C9: now also U1.64 (PC10); no longer U1.50 (PD0)
- net DB0: now also U1.27 (PB0), U6.14 (DB0); no longer U1.17 (PA0)
- net DB1: now also U1.28 (PB1), U6.15 (DB1); no longer U1.18 (PA1)
- net DB2: now also U1.29 (PB2), U6.16 (DB2); no longer U1.19 (PA2)
- net DB3: now also U1.57 (PB3), U6.17 (DB3); no longer U1.20 (PA3)
- net DB4: now also U1.58 (PB4), U6.18 (DB4); no longer U1.21 (PA4)
- net DB5: now also U1.59 (PB5), U6.19 (DB5); no longer U1.22 (PA5)
- net DB6: now also U1.60 (PB6), U6.20 (DB6); no longer U1.23 (PA6)
- net DB7: now also U1.61 (PB7), U6.21 (DB7); no longer U1.24 (PA7)
- net DC: now also U1.17 (PA0), U6.11 (D/C); no longer U1.27 (PB0)
- net ESC: now also U1.22 (PA5); no longer U1.38 (PC6)
- net GND: now also U4.5 (GND), U4.7 (T), U6.1 (GND), U6.10 (~CS), U6.33 (GND), U6.34 (LED-K1), U6.35 (LED-K2), U6.36 (LED-K3), U6.37 (LED-K4), U6.39 (GND)
- net R0: now also U1.50 (PD0); no longer U1.64 (PC10)
- net R1: now also U1.51 (PD1); no longer U1.63 (PB9)
- net R2: now also U1.52 (PD2); no longer U1.62 (PB8)
- net R3: now also U1.53 (PD3); no longer U1.61 (PB7)
- net R4: now also U1.54 (PD4); no longer U1.60 (PB6)
- net ~RD: now also U1.19 (PA2), U6.13 (~RD); no longer U1.29 (PB2)
- net ~RES: now also U1.20 (PA3), U6.30 (~RES); no longer U1.30 (PB10)
- net ~WR: now also U1.18 (PA1), U6.12 (~WR); no longer U1.28 (PB1)
- net DB11: now reaches U1.31 (PB11)
- net DB11: now also U6.25 (DB11)
- net DB12: now reaches U1.32 (PB12)
- net DB12: now also U6.26 (DB12)
- net DB13: now reaches U1.33 (PB13)
- net DB13: now also U6.27 (DB13)
- net DB14: now reaches U1.34 (PB14)
- net DB14: now also U6.28 (DB14)
- net DB15: now reaches U1.35 (PB15)
- net DB15: now also U6.29 (DB15)
- net at SW1.2 (B): now also C6.1, U4.4 (EN), U4.6 (IN)
- net +3V0: now reaches C7.1
- net +3V0: now also R1.1, U4.1 (OUT), U6.38 (LED-A), U6.7 (VDD), U6.8 (IOVDD)
- net VOUT renamed PG
- net PG: now also R1.2, U4.3 (PG); no longer C6.1
- new net DB10: U1.30 (PB10), U6.24 (DB10)
- new net DB8: U1.62 (PB8), U6.22 (DB8)
- new net DB9: U1.63 (PB9), U6.23 (DB9)
- new net IM0: U1.21 (PA4), U6.31 (IM0)
